File: hardware/RC-Sequencer.kicad_pcb (KiCad board)
At the start: 2 copper layers, 37.3 x 23.4 mm, 18 parts, among them J1 CH3, J2 Conn_02x05_Odd_Even, J3 Conn_02x04_Odd_Even, Q1 AO3400, Q2 AO3400, Q3 AO3400, Q4 AO3400, U1 ATtiny44-20SSU

Commit message: 
Parts:
- J1: value CH3 -> CH1
Changed lines of the file:
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@@
   (layers
     (0 F.Cu signal)
-    (31 B.Cu signal hide)
-    (32 B.Adhes user hide)
-    (33 F.Adhes user hide)
-    (34 B.Paste user hide)
-    (35 F.Paste user hide)
-    (36 B.SilkS user hide)
+    (31 B.Cu signal)
+    (32 B.Adhes user)
+    (33 F.Adhes user)
+    (34 B.Paste user)
+    (35 F.Paste user)
+    (36 B.SilkS user)
     (37 F.SilkS user)
-    (38 B.Mask user hide)
-    (39 F.Mask user hide)
-    (40 Dwgs.User user hide)
-    (41 Cmts.User user hide)
-    (42 Eco1.User user hide)
-    (43 Eco2.User user hide)
+    (38 B.Mask user)
+    (39 F.Mask user)
+    (40 Dwgs.User user)
+    (41 Cmts.User user)
+    (42 Eco1.User user)
+    (43 Eco2.User user)
     (44 Edge.Cuts user)
-    (45 Margin user hide)
-    (46 B.CrtYd user hide)
-    (47 F.CrtYd user hide)
-    (48 B.Fab user hide)
-    (49 F.Fab user hide)
+    (45 Margin user)
+    (46 B.CrtYd user)
+    (47 F.CrtYd user)
+    (48 B.Fab user)
+    (49 F.Fab user)
   )
   (setup
@@
       (effects (font (size 1 1) (thickness 0.15)))
     )
-    (fp_text value CH3 (at 4.385 7.35) (layer F.Fab)
+    (fp_text value CH1 (at 4.385 7.35) (layer F.Fab)
       (effects (font (size 1 1) (thickness 0.15)))
     )
@@
     )
   )
+  (dimension 23.368 (width 0.15) (layer F.Fab)
+    (gr_text "23.368 mm" (at 227.233 67.31 270) (layer F.Fab)
+      (effects (font (size 1 1) (thickness 0.15)))
+    )
+    (feature1 (pts (xy 220.98 78.994) (xy 226.519421 78.994)))
+    (feature2 (pts (xy 220.98 55.626) (xy 226.519421 55.626)))
+    (crossbar (pts (xy 225.933 55.626) (xy 225.933 78.994)))
+    (arrow1a (pts (xy 225.933 78.994) (xy 225.346579 77.867496)))
+    (arrow1b (pts (xy 225.933 78.994) (xy 226.519421 77.867496)))
+    (arrow2a (pts (xy 225.933 55.626) (xy 225.346579 56.752504)))
+    (arrow2b (pts (xy 225.933 55.626) (xy 226.519421 56.752504)))
+  )
+  (dimension 37.338 (width 0.15) (layer F.Fab)
+    (gr_text "37.338 mm" (at 202.311 49.627) (layer F.Fab)
+      (effects (font (size 1 1) (thickness 0.15)))
+    )
+    (feature1 (pts (xy 220.98 55.626) (xy 220.98 50.340579)))
+    (feature2 (pts (xy 183.642 55.626) (xy 183.642 50.340579)))
+    (crossbar (pts (xy 183.642 50.927) (xy 220.98 50.927)))
+    (arrow1a (pts (xy 220.98 50.927) (xy 219.853496 51.513421)))
+    (arrow1b (pts (xy 220.98 50.927) (xy 219.853496 50.340579)))
+    (arrow2a (pts (xy 183.642 50.927) (xy 184.768504 51.513421)))
+    (arrow2b (pts (xy 183.642 50.927) (xy 184.768504 50.340579)))
+  )
   (gr_text OUT4 (at 212.6488 72.3138) (layer B.SilkS)
     (effects (font (size 1 1) (thickness 0.15)) (justify mirror))
@@
   (gr_text JP1 (at 190.5 75.438) (layer B.SilkS)
     (effects (font (size 1 1) (thickness 0.15)) (justify mirror))
-  )
-  (dimension 23.368 (width 0.15) (layer Eco1.User)
-    (gr_text "23.368 mm" (at 226.598 67.31 270) (layer Eco1.User)
-      (effects (font (size 1 1) (thickness 0.15)))
-    )
-    (feature1 (pts (xy 220.98 78.994) (xy 225.884421 78.994)))
-    (feature2 (pts (xy 220.98 55.626) (xy 225.884421 55.626)))
-    (crossbar (pts (xy 225.298 55.626) (xy 225.298 78.994)))
-    (arrow1a (pts (xy 225.298 78.994) (xy 224.711579 77.867496)))
-    (arrow1b (pts (xy 225.298 78.994) (xy 225.884421 77.867496)))
-    (arrow2a (pts (xy 225.298 55.626) (xy 224.711579 56.752504)))
-    (arrow2b (pts (xy 225.298 55.626) (xy 225.884421 56.752504)))
-  )
-  (dimension 37.338 (width 0.15) (layer Eco1.User)
-    (gr_text "37.338 mm" (at 202.311 50.516) (layer Eco1.User)
-      (effects (font (size 1 1) (thickness 0.15)))
-    )
-    (feature1 (pts (xy 183.642 55.626) (xy 183.642 51.229579)))
-    (feature2 (pts (xy 220.98 55.626) (xy 220.98 51.229579)))
-    (crossbar (pts (xy 220.98 51.816) (xy 183.642 51.816)))
-    (arrow1a (pts (xy 183.642 51.816) (xy 184.768504 51.229579)))
-    (arrow1b (pts (xy 183.642 51.816) (xy 184.768504 52.402421)))
-    (arrow2a (pts (xy 220.98 51.816) (xy 219.853496 51.229579)))
-    (arrow2b (pts (xy 220.98 51.816) (xy 219.853496 52.402421)))
   )
   (gr_text +BAT (at 209.423 76.581) (layer B.SilkS)
@@
     (polygon
       (pts
-        (xy 207.01 53.34) (xy 207.01 81.28) (xy 223.012 81.28) (xy 223.266 53.34)
+        (xy 207.01 53.34) (xy 207.01 81.28) (xy 223.012 81.28) (xy 223.012 53.34)
       )
     )
